File: jlink-adapter/jlink-adapter.kicad_pcb (KiCad board)
At the start: 2 copper layers, 52.7 x 30.2 mm, 21 parts, among them J1 USB_C_Receptacle_USB2.0, J2 Conn_ARM_JTAG_SWD_20, J3 ESPProgJTAG_TX, J4 Conn_01x05, J5 Conn_01x06, J6 USB_A, U1 USBLC6-2SC6, U2 XC6209, U3 USBLC6-2SC6, U4 USBLC6-2SC6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

Commit message: Change layout
Connections:
- J4 pad 2: /SRST -> /SWDIO
- J4 pad 3: GND -> /SWDCLK
- J4 pad 4: /SWDIO -> GND
- J4 pad 5: /SWDCLK -> /SRST
- J5 pad 2: /TDO -> /SWDIO
- J5 pad 3: GND -> /SWDCLK
- J5 pad 4: /TDI -> /TDO
- J5 pad 5: /SWDIO -> /TDI
- J5 pad 6: /SWDCLK -> GND
Routing:
- net /TDI: track 68.2 -> 94.9 mm
- net GND: track 37.3 -> 54.5 mm, vias 5 -> 6
- net /SWDCLK: track 75.3 -> 82.6 mm
- net /SRST: track 63.6 -> 68.5 mm
- net /TDO: track 51.2 -> 47.3 mm
- net /SWDIO: track 78.8 -> 75.8 mm
