File: jlink-adapter/jlink-adapter.kicad_sch (KiCad schematic)
At the start: 21 parts, among them J1 USB_C_Receptacle_USB2.0, J2 Conn_ARM_JTAG_SWD_20, J3 ESPProgJTAG_TX, J4 Conn_01x05, J5 Conn_01x06, J6 USB_A, U1 USBLC6-2SC6, U2 XC6209, U3 USBLC6-2SC6, U4 USBLC6-2SC6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

Commit message: Add LCSC Number
Parts:
- J6: LCSC (none) -> C2345
- JP1: LCSC (none) -> 6209
- U1, U3, U4, U5: LCSC (none) -> C2827654
- U2: LCSC (none) -> C216624
Changed lines of the file:
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@@
+      (effects (font (size 1.27 1.27)) hide)
+    )
+    (property "LCSC" "C2827654" (id 4) (at 158.369 27.051 0)
       (effects (font (size 1.27 1.27)) hide)
     )
@@
     )
     (property "Datasheet" " ~" (id 3) (at 64.643 102.87 0)
+      (effects (font (size 1.27 1.27)) hide)
+    )
+    (property "LCSC" "C2345" (id 4) (at 68.453 101.6 0)
       (effects (font (size 1.27 1.27)) hide)
     )
@@
       (effects (font (size 1.27 1.27)) hide)
     )
+    (property "LCSC" "6209" (id 4) (at 24.13 17.78 0)
+      (effects (font (size 1.27 1.27)) hide)
+    )
     (pin "1")
     (pin "2")
@@
     )
     (property "Datasheet" "https://www.st.com/resource/en/datasheet/usblc6-2.pdf" (id 3) (at 65.405 124.333 0)
+      (effects (font (size 1.27 1.27)) hide)
+    )
+    (property "LCSC" "C2827654" (id 4) (at 60.325 133.223 0)
       (effects (font (size 1.27 1.27)) hide)
     )
@@
     )
     (property "Datasheet" "" (id 3) (at 115.951 95.25 0)
+      (effects (font (size 1.27 1.27)) hide)
+    )
+    (property "LCSC" "C216624" (id 4) (at 115.951 102.87 0)
       (effects (font (size 1.27 1.27)) hide)
     )
@@
       (effects (font (size 1.27 1.27)) hide)
     )
+    (property "LCSC" "C2827654" (id 4) (at 129.032 27.178 0)
+      (effects (font (size 1.27 1.27)) hide)
+    )
     (pin "1")
     (pin "2")
@@
       (effects (font (size 1.27 1.27)) hide)
     )
+    (property "LCSC" "C2827654" (id 4) (at 96.012 27.051 0)
+      (effects (font (size 1.27 1.27)) hide)
+    )

Commit message: 预备投板
Parts:
- removed D2: SMS05CT1G, Package_TO_SOT_SMD:SOT-23-6, symbol Power_Protection:ESDA6V1-5SC6
- removed U1, U3, U4, U5: USBLC6-2SC6, KisonCommon:USBLC6-2P6-SOT666, symbol Power_Protection:USBLC6-2SC6
- added R1, R4: 0, Resistor_SMD:R_0603_1608Metric, symbol Device:R
- added SW1: SW_Push, Button_Switch_SMD:SW_SPST_CK_RS282G05A3, symbol Switch:SW_Push
- added U3, U5: USBLC6-4SC6, Package_TO_SOT_SMD:SOT-23-6, symbol Power_Protection:USBLC6-4SC6
Connections:
- net DN: now also U5.6 (I/O4)
- net DP: now also U5.1 (I/O1)
- net GND: now also R1.1, U3.2 (GND), U5.2 (GND)
- net SRST: now also SW1.1, U5.3 (I/O2)
- net SWDCLK: now also U3.4 (I/O3)
- net SWDIO: now also U3.3 (I/O2)
- net TDI: now also U3.1 (I/O1)
- net TDO: now also U3.6 (I/O4)
- net VBUS: now also U3.5 (VBUS), U5.5 (VBUS)
- net VREF: now also R4.2
- new net: R1.2, R4.1, SW1.2
- no-connect marks 11 -> 8
